Commit message: Add configuration files and update URDF for TRRobot simulation in Webots

File: robocon_2027_description/urdf/tr.urdf.xacro (robot description, xacro)
@@ -7,10 +7,13 @@
   <!-- ===================================================== -->
   <xacro:property name="base_length" value="0.70"/>
-  <xacro:property name="base_width" value="0.55"/>
-  <xacro:property name="base_height" value="0.16"/>
-  <xacro:property name="wheel_radius" value="0.10"/>
+  <xacro:property name="base_width" value="0.26"/>
+  <xacro:property name="base_height" value="0.18"/>
+  <xacro:property name="upper_length" value="0.52"/>
+  <xacro:property name="upper_width" value="0.12"/>
+  <xacro:property name="upper_height" value="0.10"/>
+  <xacro:property name="wheel_radius" value="0.12"/>
   <xacro:property name="wheel_width" value="0.06"/>
-  <xacro:property name="wheel_x" value="0.23"/>
-  <xacro:property name="wheel_y" value="0.305"/>
+  <xacro:property name="wheel_x" value="0.25"/>
+  <xacro:property name="wheel_y" value="0.10"/>
   <!-- ===================================================== -->
   <!-- Material                                              -->
@@ -38,5 +41,5 @@
   <link name="base_link">
     <visual>
-      <origin xyz="0 0 0.08" rpy="0 0 0"/>
+      <origin xyz="0 0 0.09" rpy="0 0 0"/>
       <geometry>
         <box
@@ -48,5 +51,5 @@
     </visual>
     <collision>
-      <origin xyz="0 0 0.08" rpy="0 0 0"/>
+      <origin xyz="0 0 0.09" rpy="0 0 0"/>
       <geometry>
         <box
@@ -57,5 +60,5 @@
     </collision>
     <inertial>
-      <origin xyz="0 0 0.08" rpy="0 0 0"/>
+      <origin xyz="0 0 0.09" rpy="0 0 0"/>
       <mass value="12.0"/>
       <inertia
@@ -68,4 +71,30 @@
     </inertial>
   </link>
+  <link name="upper_body_link">
+    <visual>
+      <origin xyz="0 0 0.18" rpy="0 0 0"/>
+      <geometry>
+        <box
+          size="${upper_length}
+                ${upper_width}
+                ${upper_height}"/>
+      </geometry>
+      <material name="blue"/>
+    </visual>
+    <collision>
+      <origin xyz="0 0 0.18" rpy="0 0 0"/>
+      <geometry>
+        <box
+          size="${upper_length}
+                ${upper_width}
+                ${upper_height}"/>
+      </geometry>
+    </collision>
+  </link>
+  <joint name="upper_body_joint" type="fixed">
+    <parent link="base_link"/>
+    <child link="upper_body_link"/>
+    <origin xyz="0 0 0" rpy="0 0 0"/>
+  </joint>
   <!-- ===================================================== -->
   <!-- Macro roda                                            -->

File: robocon_2027_webots/urdf/tr_webots.urdf (robot description, URDF)
Before this commit: robot tr_robot, 1 links, 0 joints
Links:
- added link front_left_wheel_link; visual cylinder length=0.06 radius=0.12
- added link front_right_wheel_link; visual cylinder length=0.06 radius=0.12
- added link rear_left_wheel_link; visual cylinder length=0.06 radius=0.12
- added link rear_right_wheel_link; visual cylinder length=0.06 radius=0.12
- added link upper_body_link; collision box size=0.52 0.12 0.10; visual box size=0.52 0.12 0.10
- link base_link: geometry collision box size=0.70 0.26 0.18; visual box size=0.70 0.26 0.18
Joints:
- added joint front_left_wheel_joint: type continuous, parent base_link, child front_left_wheel_link, origin xyz=0.25 0.10 0.0 rpy=0 0 0, axis 0 1 0
- added joint front_right_wheel_joint: type continuous, parent base_link, child front_right_wheel_link, origin xyz=0.25 -0.10 0.0 rpy=0 0 0, axis 0 1 0
- added joint rear_left_wheel_joint: type continuous, parent base_link, child rear_left_wheel_link, origin xyz=-0.25 0.10 0.0 rpy=0 0 0, axis 0 1 0
- added joint rear_right_wheel_joint: type continuous, parent base_link, child rear_right_wheel_link, origin xyz=-0.25 -0.10 0.0 rpy=0 0 0, axis 0 1 0
- added joint upper_body_joint: type fixed, parent base_link, child upper_body_link, origin xyz=0 0 0 rpy=0 0 0

Commit message: mailstone 3: membuat kinematik tr robot

File: robocon_2027_description/urdf/tr.urdf.xacro (robot description, xacro)
@@ -3,107 +3,157 @@
   xmlns:xacro="http://www.ros.org/wiki/xacro"
   name="tr_robot">
-  <!-- ===================================================== -->
-  <!-- Konstanta dasar                                      -->
-  <!-- ===================================================== -->
-  <xacro:property name="base_length" value="0.70"/>
-  <xacro:property name="base_width" value="0.26"/>
-  <xacro:property name="base_height" value="0.18"/>
-  <xacro:property name="upper_length" value="0.52"/>
-  <xacro:property name="upper_width" value="0.12"/>
-  <xacro:property name="upper_height" value="0.10"/>
-  <xacro:property name="wheel_radius" value="0.12"/>
+  <!-- ==================================================== -->
+  <!-- Parameter chassis                                    -->
+  <!-- Satuan panjang: meter                                -->
+  <!-- Satuan massa: kilogram                               -->
+  <!-- ==================================================== -->
+  <xacro:property name="base_length" value="0.50"/>
+  <xacro:property name="base_width" value="0.50"/>
+  <xacro:property name="base_height" value="0.1"/>
+  <xacro:property name="base_mass" value="10.0"/>
+  <!-- ==================================================== -->
+  <!-- Parameter roda mecanum -->
+  <!-- ==================================================== -->
+  <xacro:property name="wheel_radius" value="0.10"/>
   <xacro:property name="wheel_width" value="0.06"/>
-  <xacro:property name="wheel_x" value="0.25"/>
-  <xacro:property name="wheel_y" value="0.10"/>
-  <!-- ===================================================== -->
-  <!-- Material                                              -->
-  <!-- ===================================================== -->
-  <material name="blue">
-    <color rgba="0.12 0.22 0.75 1.0"/>
+  <xacro:property name="wheel_mass" value="0.40"/>
+  <!--
+  Jarak pusat roda dari pusat robot.
+  wheel_x = setengah wheelbase depan-belakang
+  wheel_y = setengah track width kiri-kanan
+  -->
+  <xacro:property name="wheel_x" value="0.23"/>
+  <xacro:property name="wheel_y" value="0.305"/>
+  <!-- Jarak bagian bawah chassis dari lantai -->
+  <xacro:property name="ground_clearance" value="0.10"/>
+  <!-- Posisi pusat chassis terhadap base_footprint -->
+  <xacro:property
+    name="base_center_z"
+    value="${ground_clearance + base_height / 2.0}"/>
+  <xacro:property
+    name="wheel_center_z"
+    value="${ground_clearance - wheel_radius}"/>
+  <!-- ==================================================== -->
+  <!-- Parameter visual roller -->
+  <!-- ==================================================== -->
+  <xacro:property name="roller_radius" value="0.012"/>
+  <xacro:property name="roller_length" value="0.070"/>
+  <!-- ==================================================== -->
+  <!-- Material visual                                      -->
+  <!-- ==================================================== -->
+  <material name="tr_blue">
+    <color rgba="0.10 0.25 0.80 1.0"/>
   </material>
-  <material name="black">
+  <material name="wheel_black">
     <color rgba="0.03 0.03 0.03 1.0"/>
   </material>
-  <!-- ===================================================== -->
-  <!-- Base footprint                                        -->
-  <!-- ===================================================== -->
+  <material name="roller_gray">
+    <color rgba="0.30 0.30 0.30 1.0"/>
+  </material>
+  <!-- ==================================================== -->
+  <!-- Root frame -->
+  <!-- ==================================================== -->
   <link name="base_footprint"/>
-  <joint name="base_footprint_to_base_link" type="fixed">
-    <parent link="base_footprint"/>
-    <child link="base_link"/>
-    <origin
-      xyz="0 0 ${wheel_radius}"
-      rpy="0 0 0"/>
-  </joint>
-  <!-- ===================================================== -->
-  <!-- Chassis                                               -->
-  <!-- ===================================================== -->
+  <!-- ==================================================== -->
+  <!-- base_footprint                                       -->
+  <!-- Frame virtual yang berada di permukaan lantai        -->
+  <!-- ==================================================== -->
+  <!-- ==================================================== -->
+  <!-- base_link                                            -->
+  <!-- Link fisik utama robot                               -->
+  <!-- ==================================================== -->
   <link name="base_link">
     <visual>
-      <origin xyz="0 0 0.09" rpy="0 0 0"/>
+      <origin
+        xyz="0 0 0"
+        rpy="0 0 0"/>
       <geometry>
         <box
-          size="${base_length}
-                ${base_width}
-                ${base_height}"/>
+          size="${base_length} ${base_width} ${base_height}"/>
       </geometry>
-      <material name="blue"/>
+      <material name="tr_blue"/>
     </visual>
     <collision>
-      <origin xyz="0 0 0.09" rpy="0 0 0"/>
+      <origin
+        xyz="0 0 0"
+        rpy="0 0 0"/>
       <geometry>
         <box
-          size="${base_length}
-                ${base_width}
-                ${base_height}"/>
+          size="${base_length} ${base_width} ${base_height}"/>
       </geometry>
     </collision>
     <inertial>
-      <origin xyz="0 0 0.09" rpy="0 0 0"/>
-      <mass value="12.0"/>
+      <origin
+        xyz="0 0 0"
+        rpy="0 0 0"/>
+      <mass value="${base_mass}"/>
       <inertia
-        ixx="0.33"
+        ixx="${base_mass * (base_width * base_width
+              + base_height * base_height) / 12.0}"
         ixy="0.0"
         ixz="0.0"
-        iyy="0.55"
+        iyy="${base_mass * (base_length * base_length
+              + base_height * base_height) / 12.0}"
         iyz="0.0"
-        izz="0.79"/>
+        izz="${base_mass * (base_length * base_length
+              + base_width * base_width) / 12.0}"/>
     </inertial>
   </link>
-  <link name="upper_body_link">
+  <joint
+    name="base_footprint_to_base_link"
+    type="fixed">
+    <parent link="base_footprint"/>
+    <child link="base_link"/>
+    <origin xyz="0 0 ${base_center_z}" rpy="0 0 0"/>
+  </joint>
+  <!-- ==================================================== -->
+  <!-- Inertia cylinder roda -->
+  <!-- Axle roda sejajar sumbu Y -->
+  <!-- ==================================================== -->
+  <xacro:macro
+    name="mecanum_wheel_inertia"
+    params="mass radius width">
+    <inertial>
+      <origin xyz="0 0 0" rpy="0 0 0"/>
+      <mass value="${mass}"/>
+      <inertia
+        ixx="${1.0 / 12.0 * mass * (3.0 * radius * radius + width * width)}"
+        ixy="0.0"
+        ixz="0.0"
+        iyy="${1.0 / 2.0 * mass * radius * radius}"
+        iyz="0.0"
+        izz="${1.0 / 12.0 * mass * (3.0 * radius * radius + width * width)}"/>
+    </inertial>
+  </xacro:macro>
+  <!-- ==================================================== -->
+  <!-- Visual satu roller -->
+  <!-- roller_sign = +1 atau -1 menentukan kemiringan -->
+  <!-- ==================================================== -->
+  <xacro:macro
+    name="roller_visual"
+    params="x z roller_sign">
     <visual>
-      <origin xyz="0 0 0.18" rpy="0 0 0"/>
+      <origin
+        xyz="${x} 0 ${z}"
+        rpy="${pi / 2} ${roller_sign * 1.5708/2} 0"/>
       <geometry>
-        <box
-          size="${upper_length}
-                ${upper_width}
-                ${upper_height}"/>
+        <cylinder
+          radius="${roller_radius}"
+          length="${roller_length}"/>
       </geometry>
-      <material name="blue"/>
+      <material name="roller_gray"/>
     </visual>
-    <collision>
-      <origin xyz="0 0 0.18" rpy="0 0 0"/>
-      <geometry>
-        <box
-          size="${upper_length}
-                ${upper_width}
-                ${upper_height}"/>
-      </geometry>
-    </collision>
-  </link>
-  <joint name="upper_body_joint" type="fixed">
-    <parent link="base_link"/>
-    <child link="upper_body_link"/>
-    <origin xyz="0 0 0" rpy="0 0 0"/>
-  </joint>
-  <!-- ===================================================== -->
-  <!-- Macro roda                                            -->
-  <!-- ===================================================== -->
+  </xacro:macro>
+  <!-- ==================================================== -->
+  <!-- Macro roda mecanum -->
+  <!-- ==================================================== -->
   <xacro:macro
-    name="wheel"
-    params="prefix x y">
+    name="mecanum_wheel"
+    params="prefix x y z roller_sign">
     <link name="${prefix}_wheel_link">
       <visual>
-        <origin xyz="0 0 0" rpy="1.5708 0 0"/>
+        <origin
+          xyz="0 0 0"
+          rpy="${pi / 2.0} 0 0"/>
         <geometry>
           <cylinder
@@ -111,8 +161,26 @@
             length="${wheel_width}"/>
         </geometry>
-        <material name="black"/>
+        <material name="wheel_black"/>
       </visual>
+      <xacro:roller_visual
+        x="0.07"
+        z="0.07"
+        roller_sign="${roller_sign}"/>
+      <xacro:roller_visual
+        x="-0.07"
+        z="0.07"
+        roller_sign="${roller_sign}"/>
+      <xacro:roller_visual
+        x="0.07"
+        z="-0.07"
+        roller_sign="${roller_sign}"/>
+      <xacro:roller_visual
+        x="-0.07"
+        z="-0.07"
+        roller_sign="${roller_sign}"/>
       <collision>
-        <origin xyz="0 0 0" rpy="1.5708 0 0"/>
+        <origin
+          xyz="0 0 0"
+          rpy="${pi / 2.0} 0 0"/>
         <geometry>
           <cylinder
@@ -121,14 +189,8 @@
         </geometry>
       </collision>
-      <inertial>
-        <mass value="0.4"/>
-        <inertia
-          ixx="0.002"
-          ixy="0.0"
-          ixz="0.0"
-          iyy="0.002"
-          iyz="0.0"
-          izz="0.004"/>
-      </inertial>
+      <xacro:mecanum_wheel_inertia
+        mass="${wheel_mass}"
+        radius="${wheel_radius}"
+        width="${wheel_width}"/>
     </link>
     <joint
@@ -137,23 +199,48 @@
       <parent link="base_link"/>
       <child link="${prefix}_wheel_link"/>
-      <origin xyz="${x} ${y} 0" rpy="0 0 0"/>
+      <origin xyz="${x} ${y} ${z}" rpy="0 0 0"/>
       <axis xyz="0 1 0"/>
+      <dynamics
+        damping="0.01"
+        friction="0.0"/>
     </joint>
   </xacro:macro>
-  <xacro:wheel
+  <!-- ==================================================== -->
+  <!-- Joint base_footprint ke base_link                    -->
+  <!-- Tidak diberi offset karena geometry base_link sudah  -->
+  <!-- mempunyai origin sendiri terhadap frame base_link    -->
+  <!-- ==================================================== -->
+  <!-- ==================================================== -->
+  <!-- Susunan mecanum pola X -->
+  <!-- -->
+  <!-- Depan robot = +X -->
+  <!-- Kiri robot = +Y -->
+  <!-- -->
+  <!-- FL \ / FR -->
+  <!-- RL / \ RR -->
+  <!-- ==================================================== -->
+  <xacro:mecanum_wheel
     prefix="front_left"
     x="${wheel_x}"
-    y="${wheel_y}"/>
-  <xacro:wheel
+    y="${wheel_y}"
+    z="${wheel_center_z}"
+    roller_sign="-1"/>
+  <xacro:mecanum_wheel
     prefix="front_right"
     x="${wheel_x}"
-    y="${-wheel_y}"/>
-  <xacro:wheel
+    y="${-wheel_y}"
+    z="${wheel_center_z}"
+    roller_sign="1"/>
+  <xacro:mecanum_wheel
     prefix="rear_left"
     x="${-wheel_x}"
-    y="${wheel_y}"/>
-  <xacro:wheel
+    y="${wheel_y}"
+    z="${wheel_center_z}"
+    roller_sign="1"/>
+  <xacro:mecanum_wheel
     prefix="rear_right"
     x="${-wheel_x}"
-    y="${-wheel_y}"/>
+    y="${-wheel_y}"
+    z="${wheel_center_z}"
+    roller_sign="-1"/>
 </robot>
