Commit message: semangat fp nya

File: robocon_2027_webots/urdf/tr_webots.urdf (robot description, URDF)
Before this commit: robot tr_robot, 6 links, 5 joints
Links:
- removed link base_link
- removed link front_left_wheel_link
- removed link front_right_wheel_link
- removed link rear_left_wheel_link
- removed link rear_right_wheel_link
- removed link upper_body_link
Joints:
- removed joint front_left_wheel_joint
- removed joint front_right_wheel_joint
- removed joint rear_left_wheel_joint
- removed joint rear_right_wheel_joint
- removed joint upper_body_joint
